File: PCB/harp camera controller.brd (EAGLE design)
At the start: 124.5 x 80.4 mm, 113 parts, among them IC1 USBLC6-2SC6, IC10 SI8610BC-B-IS, IC2 74LVC1G240DBV, IC3 74LVC1G240DBV, IC4 FT232RL, IC5 TLV70033DDCR, IC6 ATXMEGA32A4U-AU, IC7 SN74LVC1G125DBVT, IC8 SN74LVC1G125DBVT, IC9 TLV70033DDCR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

Commit message: Updated PCB to version 1.2
Connections:
- net CLOCK_IN: now also IC6.12; no longer IC6.26
- net CLOCK_OUT: now also IC6.13; no longer IC6.27
- net U_IN_CAM2_STROBE_5V: now also IC6.27; no longer IC6.13
- net U_IN_CAM2_STROBE_PULLUP_5V: now also IC6.26; no longer IC6.12
Routing:
- net CLOCK_IN: track 53.2 -> 75.3 mm
- net CLOCK_OUT: track 30.5 -> 46.2 mm
- net U_IN_CAM2_STROBE_PULLUP_5V: track 44.7 -> 58.7 mm, vias 2 -> 4
- net U_IN_CAM2_STROBE_5V: track 45.4 -> 53.4 mm, vias 2 -> 4
- net +3V3: track 496.5 -> 491.5 mm
- net EN_CLOCK_OUT: track 33.5 -> 31.5 mm
- net U_IO_CAM1_TRIGGER: track 54.7 -> 53.6 mm
- net U_OUT0_BNC_5V: vias 4 -> 6
- net GND: vias 356 -> 353
- removed copper zone on layer 1, net N$128
- removed copper zone on layer 1, net N$159
- removed copper zone on layer 1, net N$27
Other:
- board text added: "harp camera controller v1.2"
- board text removed: "harp camera controller v1.1"

Commit message: Changed 5V output to 5.3V and released PCB v1.2
Parts:
- R12: value 31.6k -> 31.6k 0.1%
- R13: value 10k -> 10k 0.1%
Changed lines of the file:
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@@
 <attribute name="VALUE" x="15.7974" y="53.875" size="0.8128" layer="27" font="vector" ratio="15" display="off"/>
 </element>
-<element name="R12" library="rcl" package="R0402" value="31.6k" x="24.6124" y="49.5244" smashed="yes" rot="R270">
+<element name="R12" library="rcl" package="R0402" value="31.6k 0.1%" x="24.6124" y="49.5244" smashed="yes" rot="R270">
 <attribute name="DIGIKEY_PN" value="311-40.2KLRCT-ND" x="43.3068" y="49.5244" size="1.778" layer="27" rot="R270" display="off"/>
 <attribute name="MPN" value="RC0402FR-0740K2L" x="43.3068" y="49.5244" size="1.778" layer="27" rot="R270" display="off"/>
@@
 <attribute name="VALUE" x="22.7074" y="50.1594" size="1.27" layer="27" rot="R270" display="off"/>
 </element>
-<element name="R13" library="rcl" package="R0402" value="10k" x="24.6124" y="58.2988" smashed="yes" rot="R270">
+<element name="R13" library="rcl" package="R0402" value="10k 0.1%" x="24.6124" y="58.2988" smashed="yes" rot="R270">
 <attribute name="DIGIKEY_PN" value="541-3959-1-ND" x="38.43" y="64.1916" size="1.778" layer="27" rot="R270" display="off"/>
 <attribute name="MPN" value="CRCW040210K0FKED" x="38.43" y="64.1916" size="1.778" layer="27" rot="R270" display="off"/>
